File: EDID_spoofer.kicad_pcb (KiCad board)
At the start: 2 copper layers, 33 x 47.6 mm, 9 parts, among them J1 DE15_Plug_HighDensity_Mountin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, J2 DE15_Receptacle_HighDensity_M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, J3 Conn_01x04, U1 24LCS22A

Commit message: Add DDC1 ID0-3 jumpers
Allow configuration of DDC1 monitor ID bits 0-3.
Defaults to ID0 and ID2 grounded, ID1 and ID3 open -
- Color monitor which supports 1024x768.

ID1 and ID3 are shared with SDA and SCL, hence unset by default.

Also layout and signal integrity improvements.
Parts:
- added JP2: SolderJumper_2_Bridged, Jumper:SolderJumper-2_P1.3mm_Bridged_RoundedPad1.0x1.5mm, F.Cu at (25.4, 38.1)
- added JP3: SolderJumper_2_Bridged, Jumper:SolderJumper-2_P1.3mm_Bridged_RoundedPad1.0x1.5mm, F.Cu at (25.4, 50.8)
- added JP4: SolderJumper_2_Open, Jumper:SolderJumper-2_P1.3mm_Open_RoundedPad1.0x1.5mm, F.Cu at (25.4, 42.7)
- added JP5: SolderJumper_2_Open, Jumper:SolderJumper-2_P1.3mm_Open_RoundedPad1.0x1.5mm, F.Cu at (25.4, 46.7)
- moved C1 1.81 mm to (39.1, 47.8)
Connections:
- J1 pad 11: GND -> /ID0
- J1 pad 4: GND -> /ID2
Routing:
- net SDA: track 30.1 -> 55.6 mm
- net /ID0: track 0.00 -> 24.6 mm
- net /ID2: track 0.00 -> 21.4 mm
- net SCL: track 48.1 -> 67.9 mm
- net GND: track 4.34 -> 0.00 mm
- net +5V: track 42.5 -> 43.0 mm
Other:
- board text added: "ID0"
- board text added: "ID1"
- board text added: "ID2"
- board text added: "ID3"
- board text added: "JP1: Write protect [1-2] - Enabled 2-3 - Disabled DDC1 configuration: JP2: [ID0] JP3: [ID2] JP4: ID1 JP5: ID3 J1: Signal source J2: Signal sink J3: DDC2 I²C bus 1: VCC 2: SDA 3: SCL 4: GND Initial programming possible with WP set, until addres 0x7F (checksum) is set."
- board text removed: "JP1: Write protect [1-2] - Enabled 2-3 - Disabled J1: Signal source J2: Signal sink J3: DDC2 I²C bus 1: VCC 2: SDA 3: SCL 4: GND Initial programming possible with WP set, until addres 0x7F (checksum) is set."
